File: mz-pcb-guide.kicad_sch (KiCad schematic)
At the start: 21 parts

Commit message: finish matrix schema and assign footprints
Parts:
- C1, C2, C3, C4, C5, C6, C7, C8: renamed from C?; footprint (none) -> Capacitor_SMD:C_0805_2012Metric
- F1: renamed from F?; footprint (none) -> Fuse:Fuse_1206_3216Metric
- J1: renamed from J?; footprint (none) -> random-keyboard-parts:Reset_Pretty-Mask
- R1, R2, R3, R4, R5, R6: renamed from R?; footprint (none) -> Resistor_SMD:R_0805_2012Metric
- SW1: renamed from SW?; footprint (none) -> random-keyboard-parts:SKQG-1155865
- U2: renamed from U?; footprint (none) -> random-keyboard-parts:SOT143B
- USB1: renamed from USB?; footprint (none) -> Type-C:HRO-TYPE-C-31-M-12
- Y1: renamed from Y?; footprint (none) -> Crystal:Crystal_SMD_3225-4Pin_3.2x2.5mm
- gave numbers to parts that had none: 1
Other:
- added sheet matrix (matrix.kicad_sch)
- moved on the sheet: F1

Commit message: working on routing
Connections:
- net GND: now also C1.2, C2.2
- net DN: now reaches R3.1, U2.3 (IO2), USB1.5 (DN2), USB1.7 (DN1)
- net DP: now reaches R4.1, U2.2 (IO1), USB1.6 (DP1), USB1.8 (DP2)
Changed lines of the file:
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@@
   (junction (at 53.34 156.21) (diameter 0) (color 0 0 0 0)
+  )
+  (junction (at 102.87 63.5) (diameter 0) (color 0 0 0 0)
   )
   (junction (at 59.69 143.51) (diameter 0) (color 0 0 0 0)
@@
     (stroke (width 0) (type default) (color 0 0 0 0))
   )
-  (wire (pts (xy 95.25 63.5) (xy 110.49 63.5))
+  (wire (pts (xy 95.25 63.5) (xy 102.87 63.5))
     (stroke (width 0) (type default) (color 0 0 0 0))
   )
@@
     (stroke (width 0) (type default) (color 0 0 0 0))
   )
+  (wire (pts (xy 102.87 63.5) (xy 110.49 63.5))
+    (stroke (width 0) (type default) (color 0 0 0 0))
+  )
   (wire (pts (xy 63.5 130.81) (xy 66.04 130.81))
     (stroke (width 0) (type default) (color 0 0 0 0))
@@
     (stroke (width 0) (type default) (color 0 0 0 0))
   )
+  (wire (pts (xy 102.87 63.5) (xy 102.87 66.04))
+    (stroke (width 0) (type default) (color 0 0 0 0))
+  )
   (wire (pts (xy 110.49 52.07) (xy 110.49 57.15))
     (stroke (width 0) (type default) (color 0 0 0 0))
   )
-  (wire (pts (xy 102.87 60.96) (xy 102.87 66.04))
+  (wire (pts (xy 102.87 60.96) (xy 102.87 63.5))
     (stroke (width 0) (type default) (color 0 0 0 0))
   )
@@
     )
   )
+  (global_label "DN" (shape input) (at 67.945 143.51 90) (fields_autoplaced)
+    (effects (font (size 1.27 1.27)) (justify left))
+    (property "Intersheet References" "${INTERSHEET_REFS}" (id 0) (at 67.8656 138.4964 90)
+      (effects (font (size 1.27 1.27)) (justify left) hide)
+    )
+  )
   (global_label "SCK" (shape input) (at 246.38 35.56 0) (fields_autoplaced)
     (effects (font (size 1.27 1.27)) (justify left))
@@
     )
   )
+  (global_label "DP" (shape input) (at 67.945 146.05 270) (fields_autoplaced)
+    (effects (font (size 1.27 1.27)) (justify right))
+    (property "Intersheet References" "${INTERSHEET_REFS}" (id 0) (at 67.8656 151.0031 90)
+      (effects (font (size 1.27 1.27)) (justify right) hide)
+    )
+  )
