File: mz-pcb-guide.kicad_pcb (KiCad board)
At the start: 2 copper layers, 107 parts, among them J1 AVR-ISP-6, SW1 SW_Push, U1 ATmega32U4-A, U2 PRTR5V0U2X, Y1 16 MHz

Commit message: place rest of components
Parts:
- C1, C2, C3, C4, C5, C6, C7, C8, F1, J1, R1, R2, R3, R4, R5, R6, SW1, U1, U2, USB1, Y1: moved to B.Cu
- moved R6 173.8 mm to (139.5, 77.0), turned to 180 degrees
- moved U2 171.2 mm to (144.3, 78.6), turned to 180 degrees
- moved USB1 170.7 mm to (142.7, 67.4)
- moved R5 165.8 mm to (149.1, 77.0)
- moved F1 162.0 mm to (141.1, 82.4), turned to -90 degrees
- moved R1 158.4 mm to (125.9, 133.3)
- moved J1 157.9 mm to (108.4, 138.1), turned to 180 degrees
- moved SW1 136.7 mm to (121.1, 138.1), turned to 180 degrees
- moved R3 126.7 mm to (160.2, 127.0), turned to -90 degrees
- moved C3 125.4 mm to (156.8, 131.8), turned to 180 degrees
- moved R4 124.5 mm to (162.6, 127.0), turned to -90 degrees
- moved C8 123.7 mm to (153.7, 134.1), turned to 180 degrees
- moved C4 119.4 mm to (154.4, 145.3), turned to 90 degrees
- moved R2 115.6 mm to (157.6, 147.6), turned to 180 degrees
- moved C6 110.5 mm to (173.7, 134.9), turned to -90 degrees
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Other:
- board outline added: 228.6 x 81 mm

Commit message: working on routing
Parts:
- moved D31 9.62 mm to (152.5, 126.5)
- moved D40 9.46 mm to (142.8, 144.9), turned to 0 degrees
- moved C3 7.46 mm to (164.2, 130.8)
- moved U2 5.49 mm to (142.8, 83.9)
- moved F1 4.68 mm to (139.0, 86.5)
- moved D6 4.56 mm to (134.8, 89.6)
- moved C7 4.49 mm to (169.4, 131.6)
- moved C2 4.19 mm to (177.7, 138.6)
- moved R2 3.47 mm to (154.8, 145.6)
- moved C4 3.19 mm to (153.3, 142.3)
- moved C5 3.17 mm to (172.0, 145.4), turned to 90 degrees
- moved C1 2.60 mm to (177.7, 140.9)
- moved Y1 1.99 mm to (174.0, 139.7), turned to 90 degrees
- moved R5 1.67 mm to (147.5, 77.5)
- moved R6 0.89 mm to (139.6, 77.9)
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Connections:
- net Net-(R3-Pad1) renamed DN
- net Net-(R4-Pad1) renamed DP
- C1 pad 2: Net-(C1-Pad2) -> GND
- C2 pad 2: Net-(C1-Pad2) -> GND
Routing:
- net ROW3: track 0.00 -> 221.9 mm
- net ROW1: track 0.00 -> 205.1 mm
- net ROW0: track 0.00 -> 200.2 mm
- net ROW2: track 0.00 -> 198.4 mm
- net GND: track 0.00 -> 189.9 mm, vias 0 -> 6
- net +5V: track 0.00 -> 153.6 mm, vias 0 -> 6
- net DN: track 0.00 -> 73.1 mm
- net DP: track 0.00 -> 68.6 mm
- net COL5: track 0.00 -> 61.0 mm
- net COL9: track 0.00 -> 57.1 mm
- net COL2: track 0.00 -> 57.1 mm
- net COL11: track 0.00 -> 57.1 mm
- net COL10: track 0.00 -> 57.1 mm
- net COL1: track 0.00 -> 57.1 mm
- net COL0: track 0.00 -> 57.1 mm
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- added copper zone on B.Cu, net GND
- added copper zone on F.Cu, net GND

Commit message: new project subfolder
Routing:
- net +5V: track 153.6 -> 197.2 mm, vias 6 -> 7
- net GND: track 189.9 -> 207.8 mm
- net RESET: track 0.00 -> 3.98 mm
Changed lines of the file:
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@@
   (segment (start 162.779794 139.735772) (end 167.34375 144.299728) (width 0.381) (layer "B.Cu") (net 4))
   (segment (start 155.226239 144.269761) (end 158.678739 144.269761) (width 0.381) (layer "B.Cu") (net 4))
+  (segment (start 166.648772 136.40475) (end 166.438728 136.40475) (width 0.381) (layer "B.Cu") (net 4))
   (segment (start 163.28275 130.84175) (end 162.54375 131.58075) (width 0.381) (layer "B.Cu") (net 4))
   (segment (start 178.64475 138.58875) (end 177.40827 139.82523) (width 0.381) (layer "B.Cu") (net 4))
@@
   (segment (start 148.38125 77.82745) (end 149.048789 78.494989) (width 0.381) (layer "B.Cu") (net 4))
   (segment (start 168.038728 138.00475) (end 169.04375 138.00475) (width 0.381) (layer "B.Cu") (net 4))
+  (segment (start 118.00625 139.9625) (end 116.076239 141.892511) (width 0.381) (layer "B.Cu") (net 4))
   (segment (start 138.95975 77.85925) (end 138.93625 77.88275) (width 0.381) (layer "B.Cu") (net 4))
   (segment (start 159.02575 143.181728) (end 158.648772 142.80475) (width 0.381) (layer "B.Cu") (net 4))
@@
   (segment (start 177.59523 139.82523) (end 178.64475 140.87475) (width 0.381) (layer "B.Cu") (net 4))
   (segment (start 170.46623 138.00475) (end 172.58348 135.8875) (width 0.381) (layer "B.Cu") (net 4))
+  (segment (start 108.376261 141.892511) (end 107.13625 140.6525) (width 0.381) (layer "B.Cu") (net 4))
   (segment (start 161.71775 136.40475) (end 161.71775 139.735772) (width 0.381) (layer "B.Cu") (net 4))
   (segment (start 157.64375 136.40475) (end 154.961 136.40475) (width 0.381) (layer "B.Cu") (net 4))
+  (segment (start 116.076239 141.892511) (end 108.376261 141.892511) (width 0.381) (layer "B.Cu") (net 4))
   (segment (start 177.56775 137.19175) (end 178.64475 138.26875) (width 0.381) (layer "B.Cu") (net 4))
   (segment (start 161.71775 139.735772) (end 158.648772 142.80475) (width 0.381) (layer "B.Cu") (net 4))
   (segment (start 149.048789 78.494989) (end 147.793711 78.494989) (width 0.381) (layer "B.Cu") (net 4))
+  (segment (start 168.42375 131.60375) (end 168.42375 134.629772) (width 0.381) (layer "B.Cu") (net 4))
   (segment (start 144.28175 83.10175) (end 145.69075 81.69275) (width 0.381) (layer "B.Cu") (net 4))
   (segment (start 153.31075 141.32175) (end 154.79375 142.80475) (width 0.381) (layer "B.Cu") (net 4))
@@
   (segment (start 145.69075 81.69275) (end 145.69075 86.51875) (width 0.381) (layer "B.Cu") (net 4))
   (segment (start 173.6625 135.8875) (end 174.96675 137.19175) (width 0.381) (layer "B.Cu") (net 4))
+  (segment (start 168.42375 134.629772) (end 166.648772 136.40475) (width 0.381) (layer "B.Cu") (net 4))
   (segment (start 148.38125 77.50175) (end 148.38125 77.82745) (width 0.381) (layer "B.Cu") (net 4))
   (segment (start 162.54375 135.57875) (end 161.71775 136.40475) (width 0.381) (layer "B.Cu") (net 4))
@@
   (segment (start 153.92225 145.57375) (end 155.226239 144.269761) (width 0.381) (layer "B.Cu") (net 4))
   (segment (start 163.21675 130.77575) (end 163.28275 130.84175) (width 0.381) (layer "B.Cu") (net 4))
+  (segment (start 142.96025 125.95225) (end 147.21475 130.20675) (width 0.381) (layer "F.Cu") (net 5))
   (segment (start 150.64375 146.46275) (end 151.65975 147.47875) (width 0.381) (layer "F.Cu") (net 5))
-  (segment (start 139.576271 122.568271) (end 147.21475 130.20675) (width 0.381) (layer "F.Cu") (net 5))
+  (segment (start 139.576271 122.568271) (end 142.96025 125.95225) (width 0.381) (layer "F.Cu") (net 5))
   (segment (start 150.64375 130.20675) (end 154.58075 130.20675) (width 0.381) (layer "F.Cu") (net 5))
   (segment (start 147.21475 130.20675) (end 150.64375 130.20675) (width 0.381) (layer "F.Cu") (net 5))
@@
   (segment (start 139.576271 96.025271) (end 139.576271 122.568271) (width 0.381) (layer "F.Cu") (net 5))
   (via (at 154.58075 130.20675) (size 0.8) (drill 0.4) (layers "F.Cu" "B.Cu") (net 5))
+  (via (at 142.96025 125.95225) (size 0.8) (drill 0.4) (layers "F.Cu" "B.Cu") (net 5))
   (via (at 169.69375 147.47875) (size 0.8) (drill 0.4) (layers "F.Cu" "B.Cu") (net 5))
   (via (at 173.63075 130.20675) (size 0.8) (drill 0.4) (layers "F.Cu" "B.Cu") (net 5))
@@
   (via (at 138.95975 95.40875) (size 0.8) (drill 0.4) (layers "F.Cu" "B.Cu") (net 5))
   (via (at 150.64375 143.28775) (size 0.8) (drill 0.4) (layers "F.Cu" "B.Cu") (net 5))
-  (segment (start 173.6625 133.9875) (end 173.6625 130.2385) (width 0.381) (layer "B.Cu") (net 5))
+  (segment (start 124.95625 133.35) (end 132.4175 125.88875) (width 0.381) (layer "B.Cu") (net 5))
+  (segment (start 172.80525 131.60375) (end 173.6625 132.461) (width 0.381) (layer "B.Cu") (net 5))
   (segment (start 173.152 133.9875) (end 173.6625 133.9875) (width 0.381) (layer "B.Cu") (net 5))
   (segment (start 170.89775 147.47875) (end 171.97975 146.39675) (width 0.381) (layer "B.Cu") (net 5))
   (segment (start 164.14375 133.90475) (end 164.14375 132.77375) (width 0.381) (layer "B.Cu") (net 5))
+  (segment (start 173.6625 133.9875) (end 173.6625 132.461) (width 0.381) (layer "B.Cu") (net 5))
   (segment (start 166.54375 146.088761) (end 166.54375 145.30475) (width 0.381) (layer "B.Cu") (net 5))
   (segment (start 153.24475 143.28775) (end 153.31075 143.22175) (width 0.381) (layer "B.Cu") (net 5))
@@
   (segment (start 169.04375 137.20475) (end 169.93475 137.20475) (width 0.381) (layer "B.Cu") (net 5))
   (segment (start 158.678739 132.764739) (end 159.805739 132.764739) (width 0.381) (layer "B.Cu") (net 5))
+  (segment (start 109.35875 133.35) (end 124.95625 133.35) (width 0.381) (layer "B.Cu") (net 5))
   (segment (start 153.31075 143.22175) (end 153.69375 143.60475) (width 0.381) (layer "B.Cu") (net 5))
   (segment (start 150.64375 143.28775) (end 153.24475 143.28775) (width 0.381) (layer "B.Cu") (net 5))
   (segment (start 171.931739 146.444761) (end 166.89975 146.444761) (width 0.381) (layer "B.Cu") (net 5))
   (segment (start 164.14375 132.77375) (end 164.96073 131.95677) (width 0.381) (layer "B.Cu") (net 5))
+  (segment (start 107.13625 135.5725) (end 109.35875 133.35) (width 0.381) (layer "B.Cu") (net 5))
   (segment (start 153.69375 143.60475) (end 157.64375 143.60475) (width 0.381) (layer "B.Cu") (net 5))
   (segment (start 159.805739 132.764739) (end 160.14375 133.10275) (width 0.381) (layer "B.Cu") (net 5))
   (segment (start 154.6 134.14375) (end 156.18275 134.14375) (width 0.381) (layer "B.Cu") (net 5))
   (segment (start 169.93475 137.20475) (end 173.152 133.9875) (width 0.381) (layer "B.Cu") (net 5))
+  (segment (start 173.6625 132.461) (end 173.6625 130.2385) (width 0.381) (layer "B.Cu") (net 5))
   (segment (start 156.18275 134.14375) (end 157.64375 135.60475) (width 0.381) (layer "B.Cu") (net 5))
   (segment (start 173.6625 130.2385) (end 173.63075 130.20675) (width 0.381) (layer "B.Cu") (net 5))
   (segment (start 154.6 134.14375) (end 157.299728 134.14375) (width 0.381) (layer "B.Cu") (net 5))
+  (segment (start 142.89675 125.88875) (end 142.96025 125.95225) (width 0.381) (layer "B.Cu") (net 5))
   (segment (start 164.96073 131.95677) (end 165.697854 131.95677) (width 0.381) (layer "B.Cu") (net 5))
   (segment (start 157.299728 134.14375) (end 158.678739 132.764739) (width 0.381) (layer "B.Cu") (net 5))
@@
   (segment (start 166.39175 131.262874) (end 166.39175 130.20675) (width 0.381) (layer "B.Cu") (net 5))
   (segment (start 154.6 134.14375) (end 154.6 130.226) (width 0.381) (layer "B.Cu") (net 5))
+  (segment (start 170.32375 131.60375) (end 172.80525 131.60375) (width 0.381) (layer "B.Cu") (net 5))
+  (segment (start 132.4175 125.88875) (end 142.89675 125.88875) (width 0.381) (layer "B.Cu") (net 5))
   (segment (start 171.97975 146.39675) (end 171.931739 146.444761) (width 0.381) (layer "B.Cu") (net 5))
   (segment (start 166.89975 146.444761) (end 166.54375 146.088761) (width 0.381) (layer "B.Cu") (net 5))
@@
   (segment (start 141.76975 82.90175) (end 141.17675 82.90175) (width 0.381) (layer "B.Cu") (net 53))
   (segment (start 139.58477 80.71677) (end 141.76975 82.90175) (width 0.381) (layer "B.Cu") (net 53))
+  (segment (start 124.20625 136.2625) (end 124.20625 135.925) (width 0.254) (layer "B.Cu") (net 57))
+  (segment (start 124.20625 135.925) (end 126.78125 133.35) (width 0.254) (layer "B.Cu") (net 57))
   (segment (start 34.12125 118.11) (end 34.12125 137.16) (width 0.254) (layer "F.Cu") (net 58))
   (segment (start 34.12125 80.01) (end 34.12125 99.06) (width 0.254) (layer "F.Cu") (net 58))
