File: minivan/minivan.kicad_sch (KiCad schematic)
At the start: 6 parts

Commit message: finish schematic
Parts:
- added C4, C5, C6, C7: 0.1uF, Capacitor_SMD:C_0805_2012Metric, symbol Device:C_Small
- added C8: 10uF, Capacitor_SMD:C_0805_2012Metric, symbol Device:C_Small
- added F1: 500mA, Fuse:Fuse_1206_3216Metric, symbol Device:Polyfuse_Small
- added J1: AVR-ISP-6, random-keyboard-parts:Reset_Pretty-Mask, symbol Connector:AVR-ISP-6
- added R1, R2: 22, Resistor_SMD:R_0805_2012Metric, symbol Device:R_Small
- added R3, R4: 5.1k, Resistor_SMD:R_0805_2012Metric, symbol Device:R_Small
- added R6: 10k, Resistor_SMD:R_0805_2012Metric, symbol Device:R_Small
- added SW1: SW_Push, random-keyboard-parts:SKQG-1155865, symbol Switch:SW_Push
- added U1: PRTR5V0U2X, random-keyboard-parts:SOT143B, symbol random-keyboard-parts:PRTR5V0U2X
- added USB1: HRO-TYPE-C-31-M-12, Type-C:HRO-TYPE-C-31-M-12, symbol Type-C:HRO-TYPE-C-31-M-12
- C1, C2, C3: renamed from C?; footprint (none) -> Capacitor_SMD:C_0805_2012Metric
- R5: renamed from R?; footprint (none) -> Resistor_SMD:R_0805_2012Metric
- Y1: renamed from Y?; footprint (none) -> Crystal:Crystal_SMD_3225-4Pin_3.2x2.5mm
- gave numbers to parts that had none: 1
Connections:
- net +5V: now also U2.7 (VBUS), C4.1, C5.1, C6.1, C7.1, C8.1, F1.2, J1.2 (VCC), R6.1
- net D+: now also R2.2
- net D-: now also R1.2
- net GND: now also U2.15 (GND), U2.23 (GND), U2.35 (GND), U2.43 (GND), U2.5 (UGND), C4.2, C5.2, C6.2, C7.2, C8.2, J1.6 (GND), R3.2, R4.2, SW1.1, U1.1 (GND), USB1.1 (GND), USB1.12 (GND), USB1.13 (SHIELD)
- net RESET: now also J1.5 (~{RST}), R6.2, SW1.2
- net MOSI: now reaches U2.10 (PB2)
- net MOSI: now also J1.4 (MOSI)
- net MISO: now reaches U2.11 (PB3)
- net MISO: now also J1.1 (MISO)
- net col8: now reaches U2.19 (PD1)
- net col9: now reaches U2.20 (PD2)
- net col10: now reaches U2.21 (PD3)
- net col11: now reaches U2.25 (PD4)
- net col0: now reaches U2.28 (PB4)
- net col1: now reaches U2.29 (PB5)
- net col2: now reaches U2.30 (PB6)
- net col3: now reaches U2.31 (PC6)
- net col4: now reaches U2.32 (PC7)
- net col6: now reaches U2.36 (PF7)
- net col5: now reaches U2.37 (PF6)
- net row3: now reaches U2.38 (PF5)
- net row2: now reaches U2.39 (PF4)
- net row1: now reaches U2.40 (PF1)
- net row0: now reaches U2.41 (PF0)
- net col7: now reaches U2.8 (PB0)
- net SCK: now reaches U2.9 (PB1)
- net SCK: now also J1.3 (SCK)
- new net: R3.1, USB1.10 (CC2)
- new net: R4.1, USB1.4 (CC1)
- new net: R1.1, U1.3 (IO2), USB1.5 (DN2), USB1.7 (DN1)
- new net: R2.1, U1.2 (IO1), USB1.6 (DP1), USB1.8 (DP2)
- new net VCC: F1.1, U1.4 (VCC), USB1.11 (VBUS), USB1.2 (VBUS)
- no-connect marks 1 -> 9
Other:
- added sheet matrix (matrix.kicad_sch)
